File: pcb/management_pcb/management_pcb.kicad_pcb (KiCad board)
At the start: 2 copper layers, 100 x 105 mm, 25 parts, among them J1 10018783-10212TLF, J2 ATX-24, J3 Conn_02x05_Odd_Even, J4 Conn_01x04, J5 Conn_01x04, J6 Conn_01x04, M1 Fan_CPU_4pin

Commit message: Cleaded up component models, added 3d models.
Other:
- board text added: "FAN"
- board text added: "FP"
Changed lines of the file:
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@@
 		)
 		(embedded_fonts no)
+		(model "${KIPRJMOD}/parts.pretty/10018783-X0X12.stp"
+			(offset
+				(xyz 0 -1.25 0)
+			)
+			(scale
+				(xyz 1 1 1)
+			)
+			(rotate
+				(xyz -90 -0 -0)
+			)
+		)
 	)
 	(footprint "parts:SATAAPLVTK1"
@@
 		(sheetname "/")
 		(sheetfile "management_pcb.kicad_sch")
-		(units
-			(unit
-				(name "A")
-				(pins "9" "6" "7" "5" "4" "3" "1" "2" "8")
-			)
-		)
 		(attr through_hole)
 		(duplicate_pad_numbers_are_jumpers no)
@@
 			(layer "F.Fab")
 		)
+		(fp_text user "${REFERENCE}"
+			(at 0 -0.975 90)
+			(layer "F.Fab")
+			(effects
+				(font
+					(size 1.27 1.27)
+					(thickness 0.254)
+				)
+			)
+		)
 		(pad "1" thru_hole circle
 			(at 3.81 0 90)
@@
 		)
 		(embedded_fonts no)
-		(model "/home/dvogel/Downloads/sata-a-pl-vt-k-x-model.step"
+		(model "${KIPRJMOD}/parts.pretty/sata-a-pl-vt-k-x-model.step"
 			(offset
 				(xyz 8.6 -3.6 7.5)
@@
 		(sheetname "/")
 		(sheetfile "management_pcb.kicad_sch")
-		(units
-			(unit
-				(name "A")
-				(pins "9" "6" "7" "5" "4" "3" "1" "2" "8")
-			)
-		)
 		(attr through_hole)
 		(duplicate_pad_numbers_are_jumpers no)
@@
 			(layer "F.Fab")
 		)
+		(fp_text user "${REFERENCE}"
+			(at 0 -0.975 90)
+			(layer "F.Fab")
+			(effects
+				(font
+					(size 1.27 1.27)
+					(thickness 0.254)
+				)
+			)
+		)
 		(pad "1" thru_hole circle
 			(at 3.81 0 90)
@@
 		)
 		(embedded_fonts no)
-		(model "/home/dvogel/Downloads/sata-a-pl-vt-k-x-model.step"
+		(model "${KIPRJMOD}/parts.pretty/sata-a-pl-vt-k-x-model.step"
 			(offset
 				(xyz 8.6 -3.6 7.5)
@@
 		(sheetname "/")
 		(sheetfile "management_pcb.kicad_sch")
-		(units
-			(unit
-				(name "A")
-				(pins "9" "6" "7" "5" "4" "3" "1" "2" "8")
-			)
-		)
 		(attr through_hole)
 		(duplicate_pad_numbers_are_jumpers no)
@@
 			(layer "F.Fab")
 		)
+		(fp_text user "${REFERENCE}"
+			(at 0 -0.975 90)
+			(layer "F.Fab")
+			(effects
+				(font
+					(size 1.27 1.27)
+					(thickness 0.254)
+				)
+			)
+		)
 		(pad "1" thru_hole circle
 			(at 3.81 0 90)
@@
 		)
 		(embedded_fonts no)
-		(model "/home/dvogel/Downloads/sata-a-pl-vt-k-x-model.step"
+		(model "${KIPRJMOD}/parts.pretty/sata-a-pl-vt-k-x-model.step"
 			(offset
 				(xyz 8.6 -3.6 7.5)
@@
 		(sheetname "/")
 		(sheetfile "management_pcb.kicad_sch")
-		(units
-			(unit
-				(name "A")
-				(pins "9" "6" "7" "5" "4" "3" "1" "2" "8")
-			)
-		)
 		(attr through_hole)
 		(duplicate_pad_numbers_are_jumpers no)
@@
 			(layer "F.Fab")
 		)
+		(fp_text user "${REFERENCE}"
+			(at 0 -0.975 90)
+			(layer "F.Fab")
+			(effects
+				(font
+					(size 1.27 1.27)
+					(thickness 0.254)
+				)
+			)
+		)
 		(pad "1" thru_hole circle
 			(at 3.81 0 90)
@@
 		)
 		(embedded_fonts no)
-		(model "/home/dvogel/Downloads/sata-a-pl-vt-k-x-model.step"
+		(model "${KIPRJMOD}/parts.pretty/sata-a-pl-vt-k-x-model.step"
 			(offset
 				(xyz 8.6 -3.6 7.5)
@@
 		)
 		(embedded_fonts no)
-		(model "${KICAD10_3DMODEL_DIR}/Connector_Molex.3dshapes/Molex_Mini-Fit_Jr_5566-24A_2x12_P4.20mm_Vertical.step"
+		(model "${KIPRJMOD}/parts.pretty/ATX24.stp"
 			(offset
-				(xyz 0 0 0)
+				(xyz 23.1 -2.75 13)
 			)
 			(scale
@@
 			)
 			(rotate
-				(xyz 0 0 0)
+				(xyz -0 -0 -0)
 			)
 		)
@@
 			)
 			(justify left bottom)
+		)
+	)
+	(gr_text "FAN"
+		(at 17.925 12.25 0)
+		(layer "F.SilkS")
+		(effects
+			(font
+				(size 1.5 1.5)
+				(thickness 0.3)
+				(bold yes)
+			)
+			(justify left bottom)
+		)
+	)
+	(gr_text "FP"
+		(at 68.46 5.675 0)
+		(layer "F.SilkS")
+		(effects
+			(font
+				(size 1.5 1.5)
+				(thickness 0.3)
+				(bold yes)
+			)
+			(justify left bottom)

Commit message: added 3d render to readme
Other:
- board text added: "promise_pegasus_das_controller version 1"
Changed lines of the file:
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@@
 		)
+	)
+	(gr_text "promise_pegasus_das_controller\n\nversion 1"
+		(at 2.025 25.975 270)
+		(layer "F.SilkS")
+		(effects
+			(font
+				(size 1.5 1.5)
+				(thickness 0.3)
+				(bold yes)
+			)
+			(justify left bottom)
+		)
+	)
+	(barcode
+		(at 8.4 18.30625 0)
+		(layer "F.SilkS")
+		(size 13.3125 13.3125)
+		(text "https://github.com/d-vogel/promise_pegasus_das_controller")
+		(text_height 1.5)
+		(type qr)
+		(ecc_level L)
+		(hide yes)
+		(knockout no)
 	)
 	(segment

Commit message: pcb v3 [untested]. Added TMP36 temperature sensor, more GPIO exposed.
Parts:
- removed J6: Conn_01x04, Connector_Wire:SolderWire-0.1sqmm_1x04_P3.6mm_D0.4mm_OD1mm
- added U2: LM36, Package_TO_SOT_THT:TO-92_Inline, F.Cu at (48.3, 15.2)
- J5: value Conn_01x04 -> Conn_02x06_Odd_Even; footprint Connector_Wire:SolderWire-0.1sqmm_1x04_P3.6mm_D0.4mm_OD1mm -> Connector_PinHeader_2.54mm:PinHeader_2x06_P2.54mm_Vertical
- moved J2 18.8 mm to (88.4, 62.3)
- moved J5 15.6 mm to (89.8, 83.5)
Connections:
- A1 pad 1: Net-(A1-GPIO0) -> /GPIO0
- A1 pad 2: Net-(A1-GPIO1) -> /GPIO1
- A1 pad 31: unconnected-(A1-GPIO26_ADC0-Pad31)_1 -> /TEMP_SENS
- A1 pad 32: unconnected-(A1-GPIO27_ADC1-Pad32)_1 -> /GPIO27
- A1 pad 34: unconnected-(A1-GPIO28_ADC2-Pad34) -> /GPIO28
- A1 pad 4: Net-(A1-GPIO2) -> /GPIO2
- A1 pad 5: Net-(A1-GPIO3) -> /GPIO3
- A1 pad 6: Net-(A1-GPIO4) -> /GPIO4
- A1 pad 7: Net-(A1-GPIO5) -> /GPIO5
- J5 pad 1: Net-(A1-GPIO5) -> GND
- J5 pad 2: Net-(A1-GPIO4) -> GND
- J5 pad 3: Net-(A1-GPIO3) -> /GPIO0
- J5 pad 4: Net-(A1-GPIO2) -> /GPIO1
Routing:
- net /5V_STANDBY: track 98.6 -> 174.1 mm
- net /TEMP_SENS: track 0.00 -> 46.5 mm
- net /GPIO27: track 0.00 -> 39.6 mm
- net Net-(A1-GPIO5): track 38.6 -> 0.00 mm
- net /GPIO28: track 0.00 -> 37.1 mm
- net Net-(A1-GPIO4): track 36.6 -> 0.00 mm
- net Net-(A1-GPIO3): track 35.4 -> 0.00 mm
- net Net-(A1-GPIO2): track 33.8 -> 0.00 mm
- net Net-(A1-GPIO0): track 33.0 -> 0.00 mm
- net Net-(A1-GPIO1): track 28.8 -> 0.00 mm
- net /GPIO4: track 0.00 -> 24.1 mm
- net /GPIO5: track 0.00 -> 21.0 mm
- net /GPIO2: track 0.00 -> 20.0 mm
- net /GPIO3: track 0.00 -> 18.3 mm
- net /PWR_OK: track 10.6 -> 28.9 mm
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Other:
- board text added: "promise_pegasus_das_controller version 2"
- board text removed: "GPIO0"
- board text removed: "GPIO1"
- board text removed: "GPIO2"
- board text removed: "GPIO3"
- board text removed: "GPIO4"
- board text removed: "GPIO5"
- board text removed: "promise_pegasus_das_controller version 1"
