File: pcb/management_pcb/management_pcb.kicad_sch (KiCad schematic)
At the start: 25 parts, among them J1 10018783-10212TLF, J2 ATX-24, J3 Conn_02x05_Odd_Even, J4 Conn_01x04, J5 Conn_01x04, J6 Conn_01x04, M1 Fan_CPU_4pin

Commit message: pcb v3 [untested]. Added TMP36 temperature sensor, more GPIO exposed.
Parts:
- removed J5, J6: Conn_01x04, Connector_Wire:SolderWire-0.1sqmm_1x04_P3.6mm_D0.4mm_OD1mm, symbol Connector_Generic:Conn_01x04
- added J5: Conn_02x06_Odd_Even, Connector_PinHeader_2.54mm:PinHeader_2x06_P2.54mm_Vertical, symbol Connector_Generic:Conn_02x06_Odd_Even
- added U2: LM36, Package_TO_SOT_THT:TO-92_Inline, symbol Sensor_Temperature:LM35-LP
Connections:
- net 5V: now also J5.11 (Pin_11), U2.1 (+V_{S})
- net 5V_STANDBY: now also J5.12 (Pin_12)
- net GND: now also J5.1 (Pin_1), J5.2 (Pin_2), U2.3 (GND)
- net GPIO1: now reaches A1.2 (GPIO1)
- net GPIO1: now also J5.4 (Pin_4)
- net GPIO0: now reaches A1.1 (GPIO0)
- net GPIO0: now also J5.3 (Pin_3)
- net GPIO5: now reaches A1.7 (GPIO5)
- net GPIO5: now also J5.8 (Pin_8)
- net GPIO4: now reaches A1.6 (GPIO4)
- net GPIO4: now also J5.7 (Pin_7)
- net GPIO3: now reaches A1.5 (GPIO3)
- net GPIO3: now also J5.6 (Pin_6)
- net GPIO2: now reaches A1.4 (GPIO2)
- net GPIO2: now also J5.5 (Pin_5)
- net TEMP_SENS: now reaches A1.31 (GPIO26_ADC0)
- net TEMP_SENS: now also U2.2 (V_{OUT})
- net GPIO27: now reaches A1.32 (GPIO27_ADC1)
- net GPIO27: now also J5.9 (Pin_9)
- net GPIO28: now reaches A1.34 (GPIO28_ADC2)
- net GPIO28: now also J5.10 (Pin_10)
- no-connect marks 26 -> 23
